File: hardware/circuit/4E赤外線.kicad_sch (KiCad schematic)
At the start: 50 parts, among them J1 Conn_01x03_Pin, J10 SW3, J2 Conn_01x02_Pin, J3 Conn_01x03_Pin, J4 Conn_01x03_Pin, J5 赤外線, J6 motor, J7 Conn_01x03_Pin, J8 SW1, J9 SW2, Q1 IRLML6344, Q2 IRLML6344, Q3 BSS138, Q4 IRLML6402, U1 XIAO ESP32-S3 Plus / SEEED-10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, U2 L7833, U3 L7805

Commit message: kairozu kirei ni shimashita
Parts:
- C10: value C_Polarized -> 100uF
Other:
- moved on the sheet: C1, C2, C3, D2, J1, J3, J4, J6, Q2, R1, R10, R11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
